Commit message: added files to new branch for robot control

File: src/box_robot/urdf/box_robot.urdf (robot description, URDF)
Before this commit: robot pi_robot, 9 links, 8 joints
Links:
- removed link base_cylinder5
- removed link base_cylinder6
- added link base_box4, mass 1.0; collision box size=1 1.5 1; visual box size=0.15 0.2 0.1
- link base_box1: mass None -> 1.0; geometry collision box size=1 1.5 1; visual box size=0.25 0.5 0.25
- link base_box2: mass None -> 1.0; geometry collision box size=1 1.5 1; visual box size=0.15 0.15 0.8
- link base_box3: mass None -> 1.0; geometry collision box size=1 1.5 1; visual box size=0.15 0.15 0.8
- link base_cylinder1: mass None -> 50.0; geometry collision box size=1 1.5 1; visual cylinder length=0.15 radius=0.4
- link base_cylinder2: mass None -> 1.0; geometry collision box size=1 1.5 1; visual cylinder length=0.15 radius=0.3
- link base_cylinder3: mass None -> 1.0; geometry collision box size=1 1.5 1; visual cylinder length=0.1 radius=0.075
- link base_cylinder4: mass None -> 1.0; geometry collision box size=1 1.5 1; visual cylinder length=0.1 radius=0.075
Joints:
- removed joint joint8
- joint joint1: axis (none) -> 0 0 1; limit (none) -> lower=-1.57 upper=1.57 effort=10 velocity=50; origin xyz=0 0 0 rpy=0 0 0 -> xyz=0 0 0.15 rpy=0 0 0
- joint joint2: axis (none) -> 0 0 1; limit (none) -> lower=-1.57 upper=1.57 effort=100 velocity=30; origin xyz=0 0 0 rpy=0 0 0 -> xyz=0 -0.02 0.20 rpy=0 0 0; type fixed -> revolute
- joint joint3: axis (none) -> 1 0 0; child base_cylinder3 -> base_box2; limit (none) -> lower=-1.57 upper=1.57 effort=100 velocity=50; type fixed -> revolute
- joint joint4: axis (none) -> 1 0 0; child base_box2 -> base_box3; limit (none) -> lower=-1.57 upper=1.57 effort=100 velocity=100; origin xyz=0 0 0 rpy=0 0 0 -> xyz=0 0 0.8 rpy=0 0 0; parent base_cylinder3 -> base_box2; type fixed -> revolute
- joint joint5: axis (none) -> 0 1 0; child base_cylinder4 -> base_cylinder3; limit (none) -> lower=-1.57 upper=1.57 effort=100 velocity=50; origin xyz=0 0 0 rpy=0 0 0 -> xyz=0 0.7 0 rpy=0 0 0; parent base_box2 -> base_box3; type fixed -> revolute
- joint joint6: axis (none) -> 1 0 0; child base_cylinder5 -> base_box4; limit (none) -> lower=-1.57 upper=1.57 effort=100 velocity=50; parent base_cylinder4 -> base_cylinder3; type fixed -> revolute
- joint joint7: axis (none) -> 1 0 0; child base_box3 -> base_cylinder4; limit (none) -> lower=-1.57 upper=1.57 effort=10 velocity=3; parent base_cylinder5 -> base_box4

Commit message: Update box_robot.urdf

File: src/box_robot/urdf/box_robot.urdf (robot description, URDF)
Before this commit: robot pi_robot, 8 links, 7 joints
Links:
- link base_box1: mass 1.0 -> 10.0
- link base_box2: mass 1.0 -> 10.0
- link base_box3: mass 1.0 -> 10.0
- link base_cylinder1: mass 50.0 -> 300.0
- link base_cylinder2: mass 1.0 -> 10.0
- link base_cylinder3: mass 1.0 -> 5.0
Joints:
- joint joint2: limit lower=-1.57 upper=1.57 effort=100 velocity=30 -> lower=-1.57 upper=1.57 effort=100 velocity=80
- joint joint3: limit lower=-1.57 upper=1.57 effort=100 velocity=50 -> lower=-1.57 upper=1.57 effort=100 velocity=30
- joint joint4: limit lower=-1.57 upper=1.57 effort=100 velocity=100 -> lower=-1.57 upper=1.57 effort=100 velocity=50
- joint joint5: limit lower=-1.57 upper=1.57 effort=100 velocity=50 -> lower=-1.57 upper=1.57 effort=100 velocity=30
- joint joint6: limit lower=-1.57 upper=1.57 effort=100 velocity=50 -> lower=-1.57 upper=1.57 effort=100 velocity=30

Commit message: added sensor

File: src/box_robot/urdf/box_robot.urdf (robot description, URDF)
Before this commit: robot pi_robot, 8 links, 7 joints
Links:
- added link camera, mass 1.0; collision box size=1 1.5 1; visual box size=0.1 0.1 0.1
- link base_box1: mass 1.0 -> 15.0
- link base_box2: mass 1.0 -> 10
- link base_cylinder1: mass 50.0 -> 300.0
Joints:
- added joint camera_joint: type revolute, parent base_cylinder4, child camera, origin xyz=0 0.3 0 rpy=0 0 0, axis 0 0 1, limit lower=-1.57 upper=1.57 effort=100 velocity=30
- joint joint2: limit lower=-1.57 upper=1.57 effort=100 velocity=30 -> lower=-1.57 upper=1.57 effort=15 velocity=15
- joint joint3: limit lower=-1.57 upper=1.57 effort=100 velocity=50 -> lower=-1.57 upper=1.57 effort=50 velocity=50
