Commit message: give approciate name

File: src/kuka_robot/urdf/kuka.urdf (robot description, URDF)
Before this commit: robot pi_robot, 8 links, 7 joints
Joints:
- removed joint joint2
- removed joint joint3
- removed joint joint4
- removed joint joint5
- removed joint joint6
- added joint arm_twist: type revolute, parent base_box3, child base_cylinder3, origin xyz=0 0.7 0 rpy=0 0 0, axis 0 1 0, limit lower=-1.57 upper=1.57 effort=100 velocity=30
- added joint base_leg: type revolute, parent base_box1, child base_box2, origin xyz=0 0 0 rpy=0 0 0, axis 1 0 0, limit lower=-1.57 upper=1.57 effort=100 velocity=30
- added joint base_twist: type revolute, parent base_cylinder2, child base_box1, origin xyz=0 -0.02 0.20 rpy=0 0 0, axis 0 0 1, limit lower=-1.57 upper=1.57 effort=100 velocity=80
- added joint leg_to_arm: type revolute, parent base_box2, child base_box3, origin xyz=0 0 0.8 rpy=0 0 0, axis 1 0 0, limit lower=-1.57 upper=1.57 effort=100 velocity=50
- added joint tool: type revolute, parent base_cylinder3, child base_box4, origin xyz=0 0 0 rpy=0 0 0, axis 1 0 0, limit lower=-1.57 upper=1.57 effort=100 velocity=30

Commit message: splitted the kuka.urdf

File: src/kuka_robot/urdf/kuka.urdf (robot description, URDF)
Before this commit: robot pi_robot, 9 links, 8 joints
Links:
- removed link camera
Joints:
- removed joint camera_joint
